File: fmc_breakout/fmc.brd (EAGLE design)
At the start: 100 x 80 mm, 1 part

Commit message: started FMC breakout
Connections:
- new net 12V: ZED1.C35, ZED1.C37
- new net 3V3: ZED1.C39
- new net DP0-C2M_N: ZED1.C3
- new net DP0-C2M_P: ZED1.C2
- new net DP0-M2C_N: ZED1.C7
- new net DP0-M2C_P: ZED1.C6
- new net GA0: ZED1.C34
- new net GND: ZED1.C1, ZED1.C12, ZED1.C13, ZED1.C16, ZED1.C17, ZED1.C20, ZED1.C21, ZED1.C24, ZED1.C25, ZED1.C28, ZED1.C29, ZED1.C32, ZED1.C33, ZED1.C36, ZED1.C38, ZED1.C4, ZED1.C40, ZED1.C5, ZED1.C8, ZED1.C9
- new net LA06_N: ZED1.C11
- new net LA06_P: ZED1.C10
- new net LA10_N: ZED1.C15
- new net LA10_P: ZED1.C14
- new net LA14_N: ZED1.C19
- new net LA14_P: ZED1.C18
- new net LA18_N: ZED1.C23
- new net LA18_P: ZED1.C22
- new net LA27_N: ZED1.C27
- new net LA27_P: ZED1.C26
- new net SCL: ZED1.C30
- new net SDA: ZED1.C31
Changed lines of the file:
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@@
 </elements>
 <signals>
+<signal name="DP0-C2M_P">
+<contactref element="ZED1" pad="C2"/>
+</signal>
+<signal name="DP0-C2M_N">
+<contactref element="ZED1" pad="C3"/>
+</signal>
+<signal name="GND">
+<contactref element="ZED1" pad="C1"/>
+<contactref element="ZED1" pad="C4"/>
+<contactref element="ZED1" pad="C40"/>
+<contactref element="ZED1" pad="C38"/>
+<contactref element="ZED1" pad="C36"/>
+<contactref element="ZED1" pad="C33"/>
+<contactref element="ZED1" pad="C32"/>
+<contactref element="ZED1" pad="C29"/>
+<contactref element="ZED1" pad="C28"/>
+<contactref element="ZED1" pad="C21"/>
+<contactref element="ZED1" pad="C24"/>
+<contactref element="ZED1" pad="C25"/>
+<contactref element="ZED1" pad="C20"/>
+<contactref element="ZED1" pad="C16"/>
+<contactref element="ZED1" pad="C17"/>
+<contactref element="ZED1" pad="C13"/>
+<contactref element="ZED1" pad="C12"/>
+<contactref element="ZED1" pad="C9"/>
+<contactref element="ZED1" pad="C8"/>
+<contactref element="ZED1" pad="C5"/>
+<wire x1="-65.405" y1="14.605" x2="-67.945" y2="14.605" width="0" layer="19" extent="1-1"/>
+<wire x1="-62.865" y1="14.605" x2="-65.405" y2="14.605" width="0" layer="19" extent="1-1"/>
+<wire x1="-59.055" y1="14.605" x2="-62.865" y2="14.605" width="0" layer="19" extent="1-1"/>
+<wire x1="-57.785" y1="14.605" x2="-59.055" y2="14.605" width="0" layer="19" extent="1-1"/>
+<wire x1="-53.975" y1="14.605" x2="-57.785" y2="14.605" width="0" layer="19" extent="1-1"/>
+<wire x1="-52.705" y1="14.605" x2="-53.975" y2="14.605" width="0" layer="19" extent="1-1"/>
+<wire x1="-48.895" y1="14.605" x2="-52.705" y2="14.605" width="0" layer="19" extent="1-1"/>
+<wire x1="-47.625" y1="14.605" x2="-48.895" y2="14.605" width="0" layer="19" extent="1-1"/>
+<wire x1="-43.815" y1="14.605" x2="-47.625" y2="14.605" width="0" layer="19" extent="1-1"/>
+<wire x1="-42.545" y1="14.605" x2="-43.815" y2="14.605" width="0" layer="19" extent="1-1"/>
+<wire x1="-38.735" y1="14.605" x2="-42.545" y2="14.605" width="0" layer="19" extent="1-1"/>
+<wire x1="-37.465" y1="14.605" x2="-38.735" y2="14.605" width="0" layer="19" extent="1-1"/>
+<wire x1="-33.655" y1="14.605" x2="-37.465" y2="14.605" width="0" layer="19" extent="1-1"/>
+<wire x1="-32.385" y1="14.605" x2="-33.655" y2="14.605" width="0" layer="19" extent="1-1"/>
+<wire x1="-28.575" y1="14.605" x2="-32.385" y2="14.605" width="0" layer="19" extent="1-1"/>
+<wire x1="-27.305" y1="14.605" x2="-28.575" y2="14.605" width="0" layer="19" extent="1-1"/>
+<wire x1="-23.495" y1="14.605" x2="-27.305" y2="14.605" width="0" layer="19" extent="1-1"/>
+<wire x1="-22.225" y1="14.605" x2="-23.495" y2="14.605" width="0" layer="19" extent="1-1"/>
+<wire x1="-18.415" y1="14.605" x2="-22.225" y2="14.605" width="0" layer="19" extent="1-1"/>
+</signal>
+<signal name="DP0-M2C_P">
+<contactref element="ZED1" pad="C6"/>
+</signal>
+<signal name="DP0-M2C_N">
+<contactref element="ZED1" pad="C7"/>
+</signal>
+<signal name="LA06_P">
+<contactref element="ZED1" pad="C10"/>
+</signal>
+<signal name="3V3">
+<contactref element="ZED1" pad="C39"/>
+</signal>
+<signal name="12V">
+<contactref element="ZED1" pad="C37"/>
+<contactref element="ZED1" pad="C35"/>
+<wire x1="-61.595" y1="14.605" x2="-64.135" y2="14.605" width="0" layer="19" extent="1-1"/>
+</signal>
+<signal name="GA0">
+<contactref element="ZED1" pad="C34"/>
+</signal>
+<signal name="SDA">
+<contactref element="ZED1" pad="C31"/>
+</signal>
+<signal name="SCL">
+<contactref element="ZED1" pad="C30"/>
+</signal>
+<signal name="LA27_N">
+<contactref element="ZED1" pad="C27"/>
+</signal>
+<signal name="LA27_P">
+<contactref element="ZED1" pad="C26"/>
+</signal>
+<signal name="LA18_N">
+<contactref element="ZED1" pad="C23"/>
+</signal>
+<signal name="LA18_P">
+<contactref element="ZED1" pad="C22"/>
+</signal>
+<signal name="LA14_N">
+<contactref element="ZED1" pad="C19"/>
+</signal>
+<signal name="LA14_P">
+<contactref element="ZED1" pad="C18"/>
+</signal>
+<signal name="LA10_N">
+<contactref element="ZED1" pad="C15"/>
+</signal>
+<signal name="LA10_P">
+<contactref element="ZED1" pad="C14"/>
+</signal>
+<signal name="LA06_N">
+<contactref element="ZED1" pad="C11"/>
+</signal>
 </signals>
 </board>
